Commit message: upgraded to two wheel caster with no drive

File: src/ashwini/urdf/ashwini.xacro (robot description, xacro)
@@ -1,289 +1,404 @@
-<?xml version='1.0'?>
-<robot name="ashwini" xmlns:xacro="http://www.ros.org/wiki/xacro">
-	<xacro:property name="robot_name" value="ashwini" />
-	<xacro:property name="robot_chassis_mass" value="15"/>
-	<xacro:property name="robot_chassis_length" value="0.2"/>
-	<xacro:property name="robot_chassis_radius" value="0.25"/>
-	<xacro:property name="robot_caster_wheel_radius" value="0.05"/>
-	<xacro:property name="robot_caster_wheel_radius_collision" value="0.0499"/>
-	<xacro:property name="robot_wheel_mass" value="5"/>
-	<xacro:property name="robot_wheel_length" value="0.05"/>
-	<xacro:property name="robot_wheel_radius" value="0.1"/>
-	<xacro:property name="camera_mass" value="0.1"/>
-	<xacro:property name="hokoyu_mass" value="1e-5"/>
-	<!-- Make Chassis of Bot -->
-	<link name="chassis">
-		<pose>0 0 0.1 0 0 0</pose>
-		<inertial>
-			<mass value="${robot_chassis_mass}"/>
-      		<origin xyz="0.0 0 0" rpy=" 0 0 0"/>
-      		<inertia
-      			ixx="0.147116667" ixy="0" ixz="0"
-      			iyy="0.334951167" iyz="0"
-      			izz="0.3978345"
-      		/>
-		</inertial>
-		<collision name="collision">
-			<origin xyz="0 0 0.05" rpy=" 0 0 0"/>
-			<geometry>
-				<box size="0.5 0.5 0.2"/>
-			</geometry>
-		</collision>
-		<visual name="chassis_visual">
-			<origin xyz="0 0 0.05" rpy=" 0 0 0"/>
-			<geometry>
-				<box size="0.5 0.5 0.2"/>
-			</geometry>
-		</visual>
-	</link>
-	<!-- Right Wheel Back -->
-	<link name="right_wheel_back">
-		<inertial>
-			<mass value="${robot_wheel_mass}"/>
-			<origin xyz="0 0 0" rpy="0 1.5707 1.5707"/>
-			<inertia
-				ixx="0.1" ixy="0.0" ixz="0.0"
-				iyy="0.1" iyz="0.0"
-				izz="0.1"
-			/>
-		</inertial>
-		<visual>
-			<origin xyz="0 0 0" rpy="0 1.5707 1.5707"/>
-			<geometry>
-				<cylinder radius="${robot_wheel_radius}" length="${robot_wheel_length}"/>
-			</geometry>
-		</visual>
-		<collision>
-			<origin xyz="0 0 0" rpy="0 1.5707 1.5707"/>
-			<geometry>
-				<cylinder radius="${robot_wheel_radius}" length="${robot_wheel_length}"/>
-			</geometry>
-		</collision>
-	</link>
-	<!-- Right Wheel Front-->
-	<link name="right_wheel_front">
-		<inertial>
-			<mass value="${robot_wheel_mass}"/>
-			<origin xyz="0 0 0" rpy="0 1.5707 1.5707"/>
-			<inertia
-				ixx="0.1" ixy="0.0" ixz="0.0"
-				iyy="0.1" iyz="0.0"
-				izz="0.1"
-			/>
-		</inertial>
-		<visual>
-			<origin xyz="0 0 0" rpy="0 1.5707 1.5707"/>
-			<geometry>
-				<cylinder radius="${robot_wheel_radius}" length="${robot_wheel_length}"/>
-			</geometry>
-		</visual>
-		<collision>
-			<origin xyz="0 0 0" rpy="0 1.5707 1.5707"/>
-			<geometry>
-				<cylinder radius="${robot_wheel_radius}" length="${robot_wheel_length}"/>
-			</geometry>
-		</collision>
-	</link>
-	<!-- Left wheel Back-->
-	<link name="left_wheel_back">
-		<inertial>
-			<mass value="${robot_wheel_mass}"/>
-			<origin xyz="0 0 0" rpy="0 1.5707 1.5707"/>
-			<inertia
-				ixx="0.1" ixy="0.0" ixz="0.0"
-				iyy="0.1" iyz="0.0"
-				izz="0.1"
-			/>
-		</inertial>
-		<visual>
-			<origin xyz="0 0 0" rpy="0 1.5707 1.5707"/>
-			<geometry>
-				<cylinder radius="${robot_wheel_radius}" length="${robot_wheel_length}"/>
-			</geometry>
-		</visual>
-		<collision>
-			<origin xyz="0 0 0" rpy="0 1.5707 1.5707"/>
-			<geometry>
-				<cylinder radius="${robot_wheel_radius}" length="${robot_wheel_length}"/>
-			</geometry>
-		</collision>
-	</link>
-	<!-- Left wheel Front-->
-	<link name="left_wheel_front">
-		<inertial>
-			<mass value="${robot_wheel_mass}"/>
-			<origin xyz="0 0 0" rpy="0 1.5707 1.5707"/>
-			<inertia
-				ixx="0.1" ixy="0.0" ixz="0.0"
-				iyy="0.1" iyz="0.0"
-				izz="0.1"
-			/>
-		</inertial>
-		<visual>
-			<origin xyz="0 0 0" rpy="0 1.5707 1.5707"/>
-			<geometry>
-				<cylinder radius="${robot_wheel_radius}" length="${robot_wheel_length}"/>
-			</geometry>
-		</visual>
-		<collision>
-			<origin xyz="0 0 0" rpy="0 1.5707 1.5707"/>
-			<geometry>
-				<cylinder radius="${robot_wheel_radius}" length="${robot_wheel_length}"/>
-			</geometry>
-		</collision>
-	</link>
-	<!-- Camera -->
-	<link name="camera">
-		<inertial>
-			<mass value="${camera_mass}"/>
-			<origin xyz="0 0 0" rpy="0 0 0"/>
-			<inertia
-		        ixx="1e-6" ixy="0.0" ixz="0.0"
-		        iyy="1e-6" iyz="0.0"
-		        izz="1e-6"
-		      />
-		</inertial>
-		<visual>
-			<origin xyz="0 0 0" rpy="0 0 0"/>
-			<geometry>
-				<box size="0.05 0.05 0.05"/>
-			</geometry>
-		</visual>
-		<collision>
-			<origin xyz="0 0 0" rpy="0 0 0"/>
-			<geometry>
-				<box size="0.05 0.05 0.05"/>
-			</geometry>
-		</collision>
-	</link>
-	<!-- Hokuyo Lidar -->
-	<link name="hokuyo">
-		<inertial>
-			<mass value="${hokoyu_mass}"/>
-			<origin xyz="0 0 0" rpy="0 0 0"/>
-			<inertia
-		        ixx="1e-6" ixy="0.0" ixz="0.0"
-		        iyy="1e-6" iyz="0.0"
-		        izz="1e-6"
-		      />
-		</inertial>
-		<visual>
-			<origin xyz="0 0 0" rpy="0 0 0"/>
-			<geometry>
-				<mesh filename="package://ashwini/meshes/hokuyo.dae"/>
-			</geometry>
-		</visual>
-		<collision>
-			<origin xyz="0 0 0" rpy="0 0 0"/>
-			<geometry>
-				<box size="0.1 0.1 0.1"/>
-			</geometry>
-		</collision>
-	</link>
-	<!-- Project center to the ground -->
-	<link name="robot_footprint"></link>
-	<!-- Define Joints -->
-	<!-- Right Wheel Joint Back-->
-	<joint type="continuous" name="right_wheel_hinge_back">
-	    <origin xyz="-0.2 -0.30 0" rpy="0 0 0" />
-	    <parent link="chassis"/>
-	    <child link="right_wheel_back" />
-	    <axis xyz="0 1 0" rpy="0 0 0" />
-	    <limit effort="10000" velocity="1000" />
-	    <dynamics damping="1.0" friction="1.0" />
-	</joint>
-	<!-- Right Wheel Joint Front-->
-	<joint type="continuous" name="right_wheel_hinge_front">
-	    <origin xyz="0.2 -0.30 0" rpy="0 0 0" />
-	    <parent link="chassis"/>
-	    <child link="right_wheel_front" />
-	    <axis xyz="0 1 0" rpy="0 0 0" />
-	    <limit effort="10000" velocity="1000" />
-	    <dynamics damping="1.0" friction="1.0" />
-	</joint>
-	<!-- Left Wheel Joint Back-->
-	<joint type="continuous" name="left_wheel_hinge_back">
-	    <origin xyz="-0.2 0.30 0" rpy="0 0 0" />
-	    <parent link="chassis"/>
-	    <child link="left_wheel_back" />
-	    <axis xyz="0 1 0" rpy="0 0 0" />
-	    <limit effort="10000" velocity="1000" />
-	    <dynamics damping="1.0" friction="1.0" />
-	</joint>
-	<!-- Left Wheel Joint Front-->
-	<joint type="continuous" name="left_wheel_hinge_front">
-	    <origin xyz="0.2 0.30 0" rpy="0 0 0" />
-	    <parent link="chassis"/>
-	    <child link="left_wheel_front" />
-	    <axis xyz="0 1 0" rpy="0 0 0" />
-	    <limit effort="10000" velocity="1000" />
-	    <dynamics damping="1.0" friction="1.0" />
-	</joint>
-	<!-- Camera Joint -->
-	<joint name="camera_joint" type="fixed">
-		<origin xyz="0.26 0 0.4" rpy="0 0.2 0" />
-		<parent link="chassis"/>
-		<child link="camera" />
-		<axis xyz="0 1 0"/>
-	</joint>
-	<!-- Hokoyu Joint -->
-	<joint name="hokuyo_joint" type="fixed">
-	    <origin xyz="0.2 0 0.2" rpy="0 0 0" />
-	    <parent link="chassis"/>
-	    <child link="hokuyo" />
-	    <axis xyz="0 1 0"/>
-	</joint>
-	<joint name="robot_footprint_joint" type="fixed">
-		<origin xyz="0 0 0" rpy="0 0 0" />
-		<parent link="robot_footprint"/>
-		<child link="chassis" />
-	</joint>
-	<!-- Color of bot -->
-	<gazebo reference="left_wheel_front">
-		<material>Gazebo/Green</material>
-		<kp>1000000.0</kp> <!-- kp and kd for rubber -->
-		<kd>100.0</kd>
-		<mu1>1.0</mu1>
-		<mu2>1.0</mu2>
-		<maxVel>1.0</maxVel>
-		<minDepth>0.00</minDepth>
-	</gazebo>
-	<gazebo reference="left_wheel_back">
-		<material>Gazebo/Green</material>
-		<kp>1000000.0</kp> <!-- kp and kd for rubber -->
-		<kd>100.0</kd>
-		<mu1>1.0</mu1>
-		<mu2>1.0</mu2>
-		<maxVel>1.0</maxVel>
-		<minDepth>0.00</minDepth>
-	</gazebo>
-	<gazebo reference="right_wheel_front">
-		<material>Gazebo/Green</material>
-		<kp>1000000.0</kp> <!-- kp and kd for rubber -->
-		<kd>100.0</kd>
-		<mu1>1.0</mu1>
-		<mu2>1.0</mu2>
-		<maxVel>1.0</maxVel>
-		<minDepth>0.00</minDepth>
-	</gazebo>
-	<gazebo reference="right_wheel_back">
-		<material>Gazebo/Green</material>
-		<kp>1000000.0</kp> <!-- kp and kd for rubber -->
-		<kd>100.0</kd>
-		<mu1>1.0</mu1>
-		<mu2>1.0</mu2>
-		<maxVel>1.0</maxVel>
-		<minDepth>0.00</minDepth>
-	</gazebo>
-	<!--<gazebo reference="right_wheel">
-		<material>Gazebo/Green</material>
-	</gazebo>-->
-	<gazebo reference="camera">
-		<material>Gazebo/Red</material>
-	</gazebo>
-	<gazebo reference="chassis">
-		<material>Gazebo/Blue</material>
-	</gazebo>
-	<!-- Motor, Camera and Lidar Simulation -->
-	<xacro:include filename="$(find ashwini)/urdf/ashwini.gazebo" />
+<?xml version="1.0"?>
+<!--defining a namespace and the robot name are mandatory-->
+<robot name="ashwini" xmlns:xacro="ashwini_description_xacro_namespace">
+  <!--=======================================================================-->
+  <!--====================PART #0 - IMPORT FROM OTHER FILES==================-->
+  <!-- Import Rviz colors -->
+  <xacro:include filename="$(find ashwini)/urdf/materials.xacro" />
+  <!-- Import all Gazebo related items from ashwini.gazebo file -->
+  <xacro:include filename="$(find ashwini)/urdf/ashwini.gazebo" />
+  <!--==============END of PART #0 - IMPORT FROM OTHER FILES=================-->
+  <!--=======================================================================-->
+  <!--=======================================================================-->
+  <!--=========================PART #1 - CONSTANTS===========================-->
+  <!-- all the robot constants are defined in this section. Values are meters-->
+  <xacro:property name="pi" value="3.1415926535897931" />
+  <!--base link values-->
+  <xacro:property name="base_link_length_width_height" value="0.650 0.381 0.132" />
+  <xacro:property name="base_link_length" value="0.650" />
+  <xacro:property name="base_link_width" value="0.381" />
+  <xacro:property name="base_link_height" value="0.132" />
+  <xacro:property name="base_link_mass" value="20"/> <!--25 kg-->
+  <!--left and right drive wheel values (both are same size)-->
+  <xacro:property name="drive_wheel_length" value="0.049" />
+  <xacro:property name="drive_wheel_radius" value="0.181" />
+  <xacro:property name="drive_wheel_mass" value="2"/> <!--2 kg-->
+  <!--left and right castor mount plate size (both are same size)-->
+  <xacro:property name="castor_mount_link_length_width_height" value="0.1145 0.10 0.0057" />
+  <xacro:property name="castor_mount_link_length" value="0.1145" />
+  <xacro:property name="castor_mount_link_width" value="0.10" />
+  <xacro:property name="castor_mount_link_height" value="0.0057" />
+  <xacro:property name="castor_mount_link_mass" value="0.25"/> <!--0.25 kg-->
+  <!--dummy link to give castors rotation about the Z axis-->
+  <xacro:property name="castor_mount_dummy_link_length" value="0.02" />
+  <xacro:property name="castor_mount_dummy_link_width" value="0.02" />
+  <xacro:property name="castor_mount_dummy_link_height" value="0.02" />
+  <xacro:property name="castor_mount_dummy_link_mass" value="1.5"/> <!--0.25 kg-->
+  <!-- left and right castor wheels (both are same size) -->
+  <xacro:property name="castor_wheel_length" value="0.049" />
+  <xacro:property name="castor_wheel_radius" value="0.07925" />
+  <xacro:property name="castor_wheel_mass" value="2"/> <!--2 kg-->
+  <!--dimensions of shaft which is tuned by A.M.P. servo motor               -->
+  <xacro:property name="lms_rotating_shaft_length" value="0.235" />
+  <xacro:property name="lms_rotating_shaft_radius" value="0.006" />
+  <xacro:property name="lms_rotating_shaft_mass" value="1.5"/> <!--1.5 kg-->
+  <!--dimensions of plate on which the LMS sits                              -->
+  <xacro:property name="lms_plate_link_length_width_height" value="0.18415 0.1651 0.00635" />
+  <xacro:property name="lms_plate_link_length" value="0.18415" />
+  <xacro:property name="lms_plate_link_width" value="0.1651" />
+  <xacro:property name="lms_plate_link_height" value="0.00635" />
+  <xacro:property name="lms_plate_link_mass" value="0.5"/> <!--0.5 kg-->
+  <!--Box representing a collision space for the actual LMS. according to    -->
+  <!--docs, using meshes for collisions is very computationally intensive, so-->
+  <!--it is much better to define collision space as a regular box.          -->
+  <xacro:property name="lms_collision_space_length_width_height" value="0.20 0.20 0.20" />
+  <!--The dimensions of the aluminum extrusion holding the entire lms system -->
+  <xacro:property name="lms_structural_extrusion_link_length_width_height" value="0.03 0.03 0.425" />
+  <xacro:property name="lms_structural_extrusion_link_length" value="0.03" />
+  <xacro:property name="lms_structural_extrusion_link_width" value="0.03" />
+  <xacro:property name="lms_structural_extrusion_link_height" value="0.425" />
+  <xacro:property name="lms_structural_extrusion_link_mass" value="3"/> <!--3 kg-->
+  <!--Friction for joints-->
+  <xacro:property name="friction_val" value="0.15"/>
+  <!--======================END ofPART #1 - CONSTANTS========================-->
+  <!--=======================================================================-->
+  <!--=======================================================================-->
+  <!--============================PART #2 - MACROS===========================-->
+  <!-- This section contains macros for the two types of links I use, namely -->
+  <!-- box and cylinder. I do not use any spere shapes.                      -->
+  <!--&&&&&&&&&&&&&&&&&&&&&&&&&&&&&&&& BOX &&&&&&&&&&&&&&&&&&&&&&&&&&&&&&&&&&-->
+  <!-- This macro defines a box link. This makes creating a box link much    -->
+  <!-- easier and cleaner. The parameters are as follows:                    -->
+  <!-- link_name - the string that represents the link                       -->
+  <!-- length_width_height - this is the length, width and height in meters  -->
+  <!-- *origin - this is the rpy - the roll, pitch and yaw. This allows us   -->
+  <!--           to rotate the item about all 3 axis (in radians). It is     -->
+  <!--           also the xyz, which allows us to move the item along all 3  -->
+  <!--           axis from a reference point. We type this line directly in  -->
+  <!--           rather then defining 6 seperate constants per cylinder!     -->
+  <!-- material - this is the rviz color of the item                         -->
+  <!-- mass - this is the kg value of the item (estimated) to make gazebo    -->
+  <!--        happy                                                          -->
+  <xacro:macro name="box_link" params="link_name length width height material mass *origin">
+    <link name="${link_name}_link">
+      <!--If you do not explicitly specify a <collision> element. Gazebo will
+      treat your link as "invisible" to laser scanners and collision checking-->
+      <collision>
+        <geometry>
+          <box size="${length} ${width} ${height}"/>
+        </geometry>
+        <!-- line below allows us to insert:<origin rpy="${rpy}" xyz="${xyz}"/>-->
+        <xacro:insert_block name="origin" />
+      </collision>
+      <visual>
+        <geometry>
+          <!--box dimensions is Meters. L X W X H where the L X H is a ractange,
+              and the H extrudes it upwards -->
+          <box size="${length} ${width} ${height}"/>
+        </geometry>
+        <!-- line below allows us to insert:<origin rpy="${rpy}" xyz="${xyz}"/>-->
+        <xacro:insert_block name="origin" />
+        <material name="${material}"/>
+      </visual>
+      <inertial>
+        <!-- line below allows us to insert:<origin rpy="${rpy}" xyz="${xyz}"/>-->
+        <xacro:insert_block name="origin" />
+        <!--all blocks now need a 'mass' argument-->
+        <mass value="${mass}"/>
+        <!--This is the 3x3 inertial matrix. See: https://wiki.ros.org/urdf/XML/link -->
+        <!--where x=length; y=width; z=height. these lines of code came from
+        Emiliano Borghi's project-->
+        <inertia
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