Commit message: cleaned up bot

File: src/ashwini/urdf/ashwini.xacro (robot description, xacro)
@@ -1,18 +1,14 @@
 <?xml version="1.0"?>
-<!--defining a namespace and the robot name are mandatory-->
 <robot name="ashwini" xmlns:xacro="ashwini_description_xacro_namespace">
-  <!--=======================================================================-->
-  <!--====================PART #0 - IMPORT FROM OTHER FILES==================-->
-  <!-- Import Rviz colors -->
-  <xacro:include filename="$(find ashwini)/urdf/materials.xacro" />
-  <!-- Import all Gazebo related items from ashwini.gazebo file -->
+  <!-- Dummy root link without inertia -->
+  <link name="dummy_root">
+  </link>
+  <joint name="dummy_root_to_base" type="fixed">
+    <parent link="dummy_root"/>
+    <child link="base_link"/>
+    <origin xyz="0 0 0" rpy="0 0 0"/>
+  </joint>
   <xacro:include filename="$(find ashwini)/urdf/ashwini.gazebo" />
-  <!--==============END of PART #0 - IMPORT FROM OTHER FILES=================-->
-  <!--=======================================================================-->
-  <!--=======================================================================-->
-  <!--=========================PART #1 - CONSTANTS===========================-->
-  <!-- all the robot constants are defined in this section. Values are meters-->
   <xacro:property name="pi" value="3.1415926535897931" />
-  <!--base link values-->
   <xacro:property name="base_link_length_width_height" value="0.650 0.381 0.132" />
   <xacro:property name="base_link_length" value="0.650" />
@@ -20,9 +16,7 @@
   <xacro:property name="base_link_height" value="0.132" />
   <xacro:property name="base_link_mass" value="20"/> <!--25 kg-->
-  <!--left and right drive wheel values (both are same size)-->
   <xacro:property name="drive_wheel_length" value="0.049" />
   <xacro:property name="drive_wheel_radius" value="0.181" />
   <xacro:property name="drive_wheel_mass" value="2"/> <!--2 kg-->
-  <!--left and right castor mount plate size (both are same size)-->
   <xacro:property name="castor_mount_link_length_width_height" value="0.1145 0.10 0.0057" />
   <xacro:property name="castor_mount_link_length" value="0.1145" />
@@ -30,55 +24,13 @@
   <xacro:property name="castor_mount_link_height" value="0.0057" />
   <xacro:property name="castor_mount_link_mass" value="0.25"/> <!--0.25 kg-->
-  <!--dummy link to give castors rotation about the Z axis-->
   <xacro:property name="castor_mount_dummy_link_length" value="0.02" />
   <xacro:property name="castor_mount_dummy_link_width" value="0.02" />
   <xacro:property name="castor_mount_dummy_link_height" value="0.02" />
   <xacro:property name="castor_mount_dummy_link_mass" value="1.5"/> <!--0.25 kg-->
-  <!-- left and right castor wheels (both are same size) -->
   <xacro:property name="castor_wheel_length" value="0.049" />
   <xacro:property name="castor_wheel_radius" value="0.07925" />
   <xacro:property name="castor_wheel_mass" value="2"/> <!--2 kg-->
-  <!--dimensions of shaft which is tuned by A.M.P. servo motor               -->
-  <xacro:property name="lms_rotating_shaft_length" value="0.235" />
-  <xacro:property name="lms_rotating_shaft_radius" value="0.006" />
-  <xacro:property name="lms_rotating_shaft_mass" value="1.5"/> <!--1.5 kg-->
-  <!--dimensions of plate on which the LMS sits                              -->
-  <xacro:property name="lms_plate_link_length_width_height" value="0.18415 0.1651 0.00635" />
-  <xacro:property name="lms_plate_link_length" value="0.18415" />
-  <xacro:property name="lms_plate_link_width" value="0.1651" />
-  <xacro:property name="lms_plate_link_height" value="0.00635" />
-  <xacro:property name="lms_plate_link_mass" value="0.5"/> <!--0.5 kg-->
-  <!--Box representing a collision space for the actual LMS. according to    -->
-  <!--docs, using meshes for collisions is very computationally intensive, so-->
-  <!--it is much better to define collision space as a regular box.          -->
-  <xacro:property name="lms_collision_space_length_width_height" value="0.20 0.20 0.20" />
-  <!--The dimensions of the aluminum extrusion holding the entire lms system -->
-  <xacro:property name="lms_structural_extrusion_link_length_width_height" value="0.03 0.03 0.425" />
-  <xacro:property name="lms_structural_extrusion_link_length" value="0.03" />
-  <xacro:property name="lms_structural_extrusion_link_width" value="0.03" />
-  <xacro:property name="lms_structural_extrusion_link_height" value="0.425" />
-  <xacro:property name="lms_structural_extrusion_link_mass" value="3"/> <!--3 kg-->
-  <!--Friction for joints-->
   <xacro:property name="friction_val" value="0.15"/>
-  <!--======================END ofPART #1 - CONSTANTS========================-->
-  <!--=======================================================================-->
-  <!--=======================================================================-->
-  <!--============================PART #2 - MACROS===========================-->
-  <!-- This section contains macros for the two types of links I use, namely -->
-  <!-- box and cylinder. I do not use any spere shapes.                      -->
-  <!--&&&&&&&&&&&&&&&&&&&&&&&&&&&&&&&& BOX &&&&&&&&&&&&&&&&&&&&&&&&&&&&&&&&&&-->
-  <!-- This macro defines a box link. This makes creating a box link much    -->
-  <!-- easier and cleaner. The parameters are as follows:                    -->
-  <!-- link_name - the string that represents the link                       -->
-  <!-- length_width_height - this is the length, width and height in meters  -->
-  <!-- *origin - this is the rpy - the roll, pitch and yaw. This allows us   -->
-  <!--           to rotate the item about all 3 axis (in radians). It is     -->
-  <!--           also the xyz, which allows us to move the item along all 3  -->
-  <!--           axis from a reference point. We type this line directly in  -->
-  <!--           rather then defining 6 seperate constants per cylinder!     -->
-  <!-- material - this is the rviz color of the item                         -->
-  <!-- mass - this is the kg value of the item (estimated) to make gazebo    -->
-  <!--        happy                                                          -->
-  <xacro:macro name="box_link" params="link_name length width height material mass *origin">
+  <xacro:macro name="box_link" params="link_name length width height mass *origin">
     <link name="${link_name}_link">
       <!--If you do not explicitly specify a <collision> element. Gazebo will
@@ -99,5 +51,4 @@
         <!-- line below allows us to insert:<origin rpy="${rpy}" xyz="${xyz}"/>-->
         <xacro:insert_block name="origin" />
-        <material name="${material}"/>
       </visual>
       <inertial>
@@ -119,22 +70,5 @@
     </link>
   </xacro:macro>
-  <!--&&&&&&&&&&&&&&&&&&&&&&&&&&&&&&& CYLINDER &&&&&&&&&&&&&&&&&&&&&&&&&&&&&&-->
-  <!-- This macro defines a cylinder link. This makes creating a box link    -->
-  <!-- much easier and cleaner. The parameters are as follows:               -->
-  <!-- link_name - the string that represents the link                       -->
-  <!-- length - this is the length of the cylinder in meters                 -->
-  <!-- radius - the radius of the cylinder in meters                         -->
-  <!-- *origin - this is the rpy - the roll, pitch and yaw. This allows us   -->
-  <!--           to rotate the item about all 3 axis (in radians). It is     -->
-  <!--           also the xyz, which allows us to move the item along all 3  -->
-  <!--           axis from a reference point. We type this line directly in  -->
-  <!--           rather then defining 6 seperate constants per cylinder!     -->
-  <!-- material - this is the rviz color of the item                         -->
-  <!-- mass - this is the kg value of the item (estimated) to make gazebo    -->
-  <!--        happy                                                          -->
-  <!-- NOTE: the astrix means that you have to physically type the line as an-->
-  <!--       argument when using (as well as insering a xacro:insert_block...-->
-  <!--       See: https://wiki.ros.org/urdf/Tutorials/Using%20Xacro%20to%20Clean%20Up%20a%20URDF%20File#Parameterized_Macro -->
-  <xacro:macro name="cylinder_link" params="link_name length radius material mass *origin">
+  <xacro:macro name="cylinder_link" params="link_name length radius mass *origin">
     <link name="${link_name}_link">
       <!--If you do not explicitly specify a <collision> element. Gazebo will
@@ -154,5 +88,4 @@
              the 3D space relative to the origin. Note that 1.57075 is pi/2 -->
         <xacro:insert_block name="origin" />
-        <material name="${material}"/>
       </visual>
       <!--TODO-->
@@ -174,20 +107,4 @@
     </link>
   </xacro:macro>
-  <!--&&&&&&&&&&&&&&&&&&&&&&&& CONTINUOUS JOINT &&&&&&&&&&&&&&&&&&&&&&&&&&&&&-->
-  <!-- This macro defines a continuous joint. This makes creating a          -->
-  <!-- continuous joint much easier and cleaner. The parameters are as       -->
-  <!-- follows:                                                              -->
-  <!-- name - the string that represents the joint                           -->
-  <!-- rpy - the roll, pitch and yaw. This is always 0 0 0                   -->
-  <!-- xyz - this defines the axis around which the continuous joint will    -->
-  <!--       roll around.                                                    -->
-  <!-- parent - this is the parent link to which the child will connect      -->
-  <!-- child - this is the child link                                        -->
-  <!-- *origin - this is the rpy and xyz point at which the child connects to-->
-  <!--           the parent. this is entered as a block. everything is in    -->
-  <!--           meters and radians                                          -->
-  <!-- NOTE: the astrix means that you have to physically type the line as an-->
-  <!--       argument when using (as well as insering a xacro:insert_block...-->
-  <!--       See: https://wiki.ros.org/urdf/Tutorials/Using%20Xacro%20to%20Clean%20Up%20a%20URDF%20File#Parameterized_Macro -->
   <xacro:macro name="continuous_joint" params="name rpy xyz parent child friction *origin">
     <joint name="${name}_joint" type="continuous">
@@ -202,17 +119,4 @@
     </joint>
   </xacro:macro>
-  <!--&&&&&&&&&&&&&&&&&&&&&&&&&&&&& FIXED JOINT &&&&&&&&&&&&&&&&&&&&&&&&&&&&&-->
-  <!-- This macro defines a continuous joint. This makes creating a          -->
-  <!-- continuous joint much easier and cleaner. The parameters are as       -->
-  <!-- follows:                                                              -->
-  <!-- name - the string that represents the joint                           -->
-  <!-- parent - this is the parent link to which the child will connect      -->
-  <!-- child - this is the child link                                        -->
-  <!-- *origin - this is the rpy and xyz point at which the child connects to-->
-  <!--           the parent. this is entered as a block. everything is in    -->
-  <!--           meters and radians                                          -->
-  <!-- NOTE: the astrix means that you have to physically type the line as an-->
-  <!--       argument when using (as well as insering a xacro:insert_block...-->
-  <!--       See: https://wiki.ros.org/urdf/Tutorials/Using%20Xacro%20to%20Clean%20Up%20a%20URDF%20File#Parameterized_Macro -->
   <xacro:macro name="fixed_joint" params="name parent child *origin">
     <joint name="${name}_joint" type="fixed">
@@ -223,18 +127,11 @@
     </joint>
   </xacro:macro>
-  <!--======================END ofPART #2 - MACROS===========================-->
-  <!--=======================================================================-->
-  <!--=======================================================================-->
-  <!--===================PART #3 - LINK & JOINT DEFINITIONS==================-->
-  <!-- all the robot constants are defined in this section. Values are meters-->
-  <!--base_link is the parent link onto which all other links join to -->
   <xacro:box_link link_name="base" length="${base_link_length}"
                                    width="${base_link_width}"
-                                   height="${base_link_height}" material="white" mass="${base_link_mass}">
+                                   height="${base_link_height}"  mass="${base_link_mass}">
     <!--origin rpy="0 0 0" xyz="-0.325 -0.1905 0.066"/-->
     <origin rpy="0 0 0" xyz="-0.325 -0.1905 0.066"/>
   </xacro:box_link>
-  <!--left_drive_wheel_link is a well named link :-) -->
-  <xacro:cylinder_link link_name="left_drive_wheel" length="${drive_wheel_length}" radius="${drive_wheel_radius}" material="black" mass="${drive_wheel_mass}">
+  <xacro:cylinder_link link_name="left_drive_wheel" length="${drive_wheel_length}" radius="${drive_wheel_radius}"  mass="${drive_wheel_mass}">
     <origin xyz="0 0 0" rpy="${pi/2} 0 0"/>
   </xacro:cylinder_link>
@@ -245,5 +142,5 @@
   </xacro:continuous_joint>
   <!--right_drive_wheel_link is a well named link :-) -->
-  <xacro:cylinder_link link_name="right_drive_wheel" length="${drive_wheel_length}" radius="${drive_wheel_radius}" material="black" mass="${drive_wheel_mass}">
+  <xacro:cylinder_link link_name="right_drive_wheel" length="${drive_wheel_length}" radius="${drive_wheel_radius}"  mass="${drive_wheel_mass}">
     <origin xyz="0 0 0" rpy="${pi/2} 0 0"/>
   </xacro:cylinder_link>
@@ -257,5 +154,5 @@
   <xacro:box_link link_name="left_castor_mount" length="${castor_mount_link_length}"
                                                 width="${castor_mount_link_width}"
-                                                height="${castor_mount_link_height}" material="white"
+                                                height="${castor_mount_link_height}"
                                                 mass="${castor_mount_link_mass}">
     <origin xyz="0 0 0" rpy="0 0 0" />
@@ -268,5 +165,5 @@
   <xacro:box_link link_name="left_castor_dummy" length="${castor_mount_dummy_link_length}"
                                                 width="${castor_mount_dummy_link_width}"
-                                                height="${castor_mount_dummy_link_height}" material="white"
+                                                height="${castor_mount_dummy_link_height}"
                                                 mass="${castor_mount_dummy_link_mass}">
     <origin xyz="0 0 0" rpy="0 0 0" />
@@ -278,5 +175,5 @@
   </xacro:continuous_joint>
   <!--left_castor_wheel_link is a well named link :-) -->
-  <xacro:cylinder_link link_name="left_castor_wheel" length="${castor_wheel_length}" radius="${castor_wheel_radius}" material="Black" mass="${castor_wheel_mass}">
+  <xacro:cylinder_link link_name="left_castor_wheel" length="${castor_wheel_length}" radius="${castor_wheel_radius}"  mass="${castor_wheel_mass}">
     <origin xyz="0 0 0" rpy="${pi/2} 0 0"/>
   </xacro:cylinder_link>
@@ -290,5 +187,5 @@
   <xacro:box_link link_name="right_castor_mount" length="${castor_mount_link_length}"
                                                  width="${castor_mount_link_width}"
-                                                 height="${castor_mount_link_height}" material="black"
+                                                 height="${castor_mount_link_height}"
                                                  mass="${castor_mount_link_mass}">
     <origin xyz="0 0 0" rpy="0 0 0" />
@@ -301,5 +198,5 @@
   <xacro:box_link link_name="right_castor_dummy" length="${castor_mount_dummy_link_length}"
                                                  width="${castor_mount_dummy_link_width}"
-                                                 height="${castor_mount_dummy_link_height}" material="orange"
+                                                 height="${castor_mount_dummy_link_height}"
                                                  mass="${castor_mount_dummy_link_mass}">
     <origin xyz="0 0 0" rpy="0 0 0" />
@@ -312,5 +209,5 @@
   <!--right_castor_wheel_link is a well named link :-) -->
   <xacro:cylinder_link link_name="right_castor_wheel" length="${castor_wheel_length}" radius="${castor_wheel_radius}"
-                       material="Black" mass="${castor_wheel_mass}">
+                        mass="${castor_wheel_mass}">
     <origin xyz="0 0 0" rpy="${pi/2} 0 0"/>
   </xacro:cylinder_link>
@@ -320,85 +217,3 @@
     <origin xyz="-0.037 0 -0.10785"/>
   </xacro:continuous_joint>
-  <!--lms_structrual_extrusion is the aluminum extrusion that is supporting   -->
-  <!-- the entire LMS structure. I put it here for aestetics.                -->
-  <xacro:box_link link_name="lms_structural_extrusion" length="${lms_structural_extrusion_link_length}"
-                                                      width="${lms_structural_extrusion_link_width}"
-                                                      height="${lms_structural_extrusion_link_height}" material="white" mass="${lms_structural_extrusion_link_mass}">
-    <origin xyz="0 0 0" rpy="0 0 0" />
-  </xacro:box_link>
-  <!--    -->
-  <xacro:fixed_joint name="base_link_to_lms_structural_extrusion" parent="base" child="lms_structural_extrusion">
-    <origin xyz="-0.3531 -0.1905 0.2173"/>
-  </xacro:fixed_joint>
-  <!--This is the rotating shaft on which the LMS sits, and which the servo  -->
-  <!--motor rotates.                                                         -->
-  <xacro:cylinder_link link_name="lms_rotating_shaft" length="${lms_rotating_shaft_length}" radius="${lms_rotating_shaft_radius}" material="white" mass="${lms_rotating_shaft_mass}">
-    <origin xyz="0 0 0" rpy="0 0 0"/>
-  </xacro:cylinder_link>
-  <!-- This joint attaches the rotating_lms_shaft to the base link -->
-  <xacro:continuous_joint name="base_link_to_rotating_lms_shaft" rpy="0 0 0" xyz="0 0 1"
-                          parent="base" child="lms_rotating_shaft" friction="${friction_val}">
-    <origin xyz="-0.2531 -0.1905 0.3195"/>
-  </xacro:continuous_joint>
-  <!--lms_plate is the plate onto which I mounted the lms :-) -->
-  <xacro:box_link link_name="lms_plate" length="${lms_plate_link_length}"
-                                        width="${lms_plate_link_width}"
-                                        height="${lms_plate_link_height}" material="white" mass="${lms_plate_link_mass}">
-    <origin xyz="0 0 0" rpy="0 0 0" />
-  </xacro:box_link>
-   <!-- -->
-  <xacro:fixed_joint name="lms_rotating_shaft_to_lms_plate" parent="lms_rotating_shaft" child="lms_plate">
-    <origin xyz="-0.04905 0 0.120675"/>
-  </xacro:fixed_joint>
-  <!--=======================================================================-->
-  <!--========SPECIAL CASES for LINK & JOINT DEFINITIONS=====================-->
-  <!-- This area contains one offs, such as a link with meshes, a links that -->
-  <!-- anchor the laser (point in space from which all /scan topic data is   -->
-  <!-- refrenced), and I think thats it. But basically a bunch of non xacro  -->
-  <!-- code (even though where I can, I still use xacro. Ex: joints).        -->
-  <!--=======================================================================-->
-  <joint name="lms_plate_to_lms_mesh" type="fixed">
-	<!--axis tag is not used according to: https://wiki.ros.org/urdf/XML/joint -->
-    <!--axis xyz="0 0 0" /-->
-	<!--relationship of child link to parent link. This is doing the laser rendering
-        in rviz, not the mesh.-->
-    <origin xyz=".15 0 .1" rpy="-1.57 0.0 0"/>
-    <parent link="lms_plate_link"/>
-    <child link="laser"/>
-  </joint>
-  <!-- this link is the actual LMS, and is rendered by importing a mesh file.-->
-  <!-- This link definition is not using any macros as there is only one type-->
-  <!-- of this link. No need to automate it.                                 -->
-  <link name="laser">
-    <collision>
-      <origin rpy="0 0 0" xyz="0 0 0"/>
-	  <geometry>
-        <box size="${lms_collision_space_length_width_height}"/>
-      </geometry>
-    </collision>
-    <visual>
-      <geometry>
-        <!--The meshes file was demonstrated by the tutorial. The sizing was
-            figured out by my question on answers.ros.org. the values are
-            multipliers. We are showing the size at 9.5% of the original mesh file -->
-        <mesh filename="package://ashwini/meshes/lms-200-30106.dae" scale="0.095 0.095 0.095"/>
-      </geometry>
-	  <!--This is responsible for rendering the mesh on the lms plate-->
-      <origin rpy="1.57 0.0 0.0" xyz="-0.02 0.025 0"/>
-      <material name="white"/>
-    </visual>
-    <inertial>
-      <origin rpy="0 0 0" xyz="0 0 0"/>
-      <!--mass is the kg value of the link-->
-      <mass value="1"/>
-      <!--3x3 inertia matrix. See: https://wiki.ros.org/urdf/XML/link
-      the values are copy pasted from: http://gazebosim.org/tutorials/?tut=ros_urdf-->
-      <inertia
-        ixx="1.0" ixy="0.0" ixz="0.0"
-        iyy="1.0" iyz="0.0"
-        izz="1.0"/>
-    </inertial>
-  </link>
-  <!--===============END OF PART #3 - LINK & JOINT DEFINITIONS===============-->
-  <!--=======================================================================-->
 </robot>
