Commit message: proper bot

File: src/ashwini/urdf/ashwini.xacro (robot description, xacro)
@@ -62,10 +62,10 @@
         <inertia
           ixx="${mass*(width*width+height*height)/12}"
-    	  ixy = "0"
-    	  ixz = "0"
-    	  iyy="${mass*(length*length+height*height)/12}"
-    	  iyz = "0"
-    	  izz="${mass*(length*length+height*height)/12}"/>
-      </inertial>
+          ixy = "0"
+          ixz = "0"
+          iyy="${mass*(length*length+height*height)/12}"
+          iyz = "0"
+          izz="${mass*(length*length+height*height)/12}"/>
+        </inertial>
     </link>
   </xacro:macro>
@@ -139,5 +139,5 @@
   <xacro:continuous_joint name="base_to_left_drive_wheel" rpy="0 0 0" xyz="0 1 0" parent="base" child="left_drive_wheel"
                           friction="${friction_val}">
-    <origin xyz="-0.52835 0.037 -0.035"/>
+    <origin xyz="-0.05 0.037 -0.035"/>
   </xacro:continuous_joint>
   <!--right_drive_wheel_link is a well named link :-) -->
@@ -148,5 +148,5 @@
   <xacro:continuous_joint name="base_to_right_drive_wheel" rpy="0 0 0" xyz="0 1 0" parent="base" child="right_drive_wheel"
                           friction="${friction_val}">
-    <origin xyz="-0.52835 -0.421 -0.035"/>
+    <origin xyz="-0.05 -0.421 -0.035"/>
   </xacro:continuous_joint>
   <!--+++++++++++++++++++++++++++++++++++LEFT CASTOR+++++++++++++++++++++++++++++++++++++++++++++++++++-->
@@ -160,5 +160,5 @@
    <!--joint-->
   <xacro:fixed_joint name="base_to_left_castor_mount" parent="base" child="left_castor_mount">
-    <origin xyz="-0.09445 -0.041 -0.03265"/>
+    <origin xyz="-0.52835 -0.041 -0.03265"/>
   </xacro:fixed_joint>
   <!--left_caster_dummy to give the castor wheel rotation about the Z axis -->
@@ -193,5 +193,5 @@
    <!--        -->
   <xacro:fixed_joint name="base_to_right_castor_mount" parent="base" child="right_castor_mount">
-    <origin xyz="-0.09445 -0.344 -0.03265"/>
+    <origin xyz="-0.52835 -0.344 -0.03265"/>
   </xacro:fixed_joint>
   <!--right_caster_dummy to give the castor wheel rotation about the Z axis -->

Commit message: imu added

File: src/ashwini/urdf/ashwini.xacro (robot description, xacro)
@@ -11,4 +11,6 @@
   <xacro:include filename="$(find ashwini)/urdf/ashwini.gazebo" />
   <xacro:property name="pi" value="3.1415926535897931" />
+  <xacro:property name="camera_mass" value="0.1"/>
+	<xacro:property name="hokoyu_mass" value="1e-5"/>
   <xacro:property name="base_link_length_width_height" value="0.650 0.381 0.132" />
   <xacro:property name="base_link_length" value="0.650" />
@@ -217,3 +219,91 @@
     <origin xyz="-0.037 0 -0.10785"/>
   </xacro:continuous_joint>
+  <link name="camera">
+		<inertial>
+			<mass value="${camera_mass}"/>
+			<origin xyz="0 0 0" rpy="0 0 0"/>
+			<inertia
+		        ixx="1e-6" ixy="0.0" ixz="0.0"
+		        iyy="1e-6" iyz="0.0"
+		        izz="1e-6"
+		      />
+		</inertial>
+		<visual>
+			<origin xyz="0 0 0" rpy="0 0 0"/>
+			<geometry>
+				<box size="0.05 0.05 0.05"/>
+			</geometry>
+		</visual>
+		<collision>
+			<origin xyz="0 0 0" rpy="0 0 0"/>
+			<geometry>
+				<box size="0.05 0.05 0.05"/>
+			</geometry>
+		</collision>
+	</link>
+  <link name="hokuyo">
+		<inertial>
+			<mass value="${hokoyu_mass}"/>
+			<origin xyz="0 0 0" rpy="0 0 0"/>
+			<inertia
+		        ixx="1e-6" ixy="0.0" ixz="0.0"
+		        iyy="1e-6" iyz="0.0"
+		        izz="1e-6"
+		      />
+		</inertial>
+		<visual>
+			<origin xyz="0 0 0" rpy="0 0 0"/>
+			<geometry>
+				<mesh filename="package://atom/meshes/hokuyo.dae"/>
+			</geometry>
+		</visual>
+		<collision>
+			<origin xyz="0 0 0" rpy="0 0 0"/>
+			<geometry>
+				<box size="0.1 0.1 0.1"/>
+			</geometry>
+		</collision>
+	</link>
+  <joint name="camera_joint" type="fixed">
+		<origin xyz="0.006 -0.2 0.4" rpy="0 0.2 0" />
+		<parent link="base_link"/>
+		<child link="camera" />
+		<axis xyz="0 1 0"/>
+	</joint>
+	<!-- Hokoyu Joint -->
+	<joint name="hokuyo_joint" type="fixed">
+	    <origin xyz="0.001 -0.2 0.2" rpy="0 0 0" />
+	    <parent link="base_link"/>
+	    <child link="hokuyo" />
+	    <axis xyz="0 1 0"/>
+	</joint>
+    <!-- IMU Sensor -->
+  <link name="imu_link">
+    <inertial>
+      <mass value="0.05"/>
+      <origin xyz="0 0 0" rpy="0 0 0"/>
+      <inertia ixx="0.0001" ixy="0.0" ixz="0.0"
+               iyy="0.0001" iyz="0.0"
+               izz="0.0001"/>
+    </inertial>
+    <visual>
+      <geometry>
+        <box size="0.05 0.05 0.02"/>
+      </geometry>
+      <material name="Blue">
+        <color rgba="0.0 0.0 1.0 1.0"/>
+      </material>
+    </visual>
+    <collision>
+      <geometry>
+        <box size="0.05 0.05 0.02"/>
+      </geometry>
+    </collision>
+  </link>
+  <!-- IMU Joint (Attach to Base Link) -->
+  <joint name="imu_joint" type="fixed">
+    <parent link="base_link"/>
+    <child link="imu_link"/>
+    <origin xyz="-0.2 -0.2 0.144" rpy="0 0 0"/>
+  </joint>
 </robot>

Commit message: shifted to custom planner

File: src/ashwini/urdf/ashwini.xacro (robot description, xacro)
@@ -11,4 +11,6 @@
   <xacro:include filename="$(find ashwini)/urdf/ashwini.gazebo" />
   <xacro:property name="pi" value="3.1415926535897931" />
+  <xacro:property name="camera_mass" value="0.1"/>
+	<xacro:property name="hokoyu_mass" value="1e-5"/>
   <xacro:property name="base_link_length_width_height" value="0.650 0.381 0.132" />
   <xacro:property name="base_link_length" value="0.650" />
@@ -62,10 +64,10 @@
         <inertia
           ixx="${mass*(width*width+height*height)/12}"
-    	  ixy = "0"
-    	  ixz = "0"
-    	  iyy="${mass*(length*length+height*height)/12}"
-    	  iyz = "0"
-    	  izz="${mass*(length*length+height*height)/12}"/>
-      </inertial>
+          ixy = "0"
+          ixz = "0"
+          iyy="${mass*(length*length+height*height)/12}"
+          iyz = "0"
+          izz="${mass*(length*length+height*height)/12}"/>
+        </inertial>
     </link>
   </xacro:macro>
@@ -139,5 +141,5 @@
   <xacro:continuous_joint name="base_to_left_drive_wheel" rpy="0 0 0" xyz="0 1 0" parent="base" child="left_drive_wheel"
                           friction="${friction_val}">
-    <origin xyz="-0.52835 0.037 -0.035"/>
+    <origin xyz="-0.05 0.037 -0.035"/>
   </xacro:continuous_joint>
   <!--right_drive_wheel_link is a well named link :-) -->
@@ -148,5 +150,5 @@
   <xacro:continuous_joint name="base_to_right_drive_wheel" rpy="0 0 0" xyz="0 1 0" parent="base" child="right_drive_wheel"
                           friction="${friction_val}">
-    <origin xyz="-0.52835 -0.421 -0.035"/>
+    <origin xyz="-0.05 -0.421 -0.035"/>
   </xacro:continuous_joint>
   <!--+++++++++++++++++++++++++++++++++++LEFT CASTOR+++++++++++++++++++++++++++++++++++++++++++++++++++-->
@@ -160,5 +162,5 @@
    <!--joint-->
   <xacro:fixed_joint name="base_to_left_castor_mount" parent="base" child="left_castor_mount">
-    <origin xyz="-0.09445 -0.041 -0.03265"/>
+    <origin xyz="-0.52835 -0.041 -0.03265"/>
   </xacro:fixed_joint>
   <!--left_caster_dummy to give the castor wheel rotation about the Z axis -->
@@ -193,5 +195,5 @@
    <!--        -->
   <xacro:fixed_joint name="base_to_right_castor_mount" parent="base" child="right_castor_mount">
-    <origin xyz="-0.09445 -0.344 -0.03265"/>
+    <origin xyz="-0.52835 -0.344 -0.03265"/>
   </xacro:fixed_joint>
   <!--right_caster_dummy to give the castor wheel rotation about the Z axis -->
@@ -217,3 +219,91 @@
     <origin xyz="-0.037 0 -0.10785"/>
   </xacro:continuous_joint>
+  <link name="camera">
+		<inertial>
+			<mass value="${camera_mass}"/>
+			<origin xyz="0 0 0" rpy="0 0 0"/>
+			<inertia
+		        ixx="1e-6" ixy="0.0" ixz="0.0"
+		        iyy="1e-6" iyz="0.0"
+		        izz="1e-6"
+		      />
+		</inertial>
+		<visual>
+			<origin xyz="0 0 0" rpy="0 0 0"/>
+			<geometry>
+				<box size="0.05 0.05 0.05"/>
+			</geometry>
+		</visual>
+		<collision>
+			<origin xyz="0 0 0" rpy="0 0 0"/>
+			<geometry>
+				<box size="0.05 0.05 0.05"/>
+			</geometry>
+		</collision>
+	</link>
+  <link name="hokuyo">
+		<inertial>
+			<mass value="${hokoyu_mass}"/>
+			<origin xyz="0 0 0" rpy="0 0 0"/>
+			<inertia
+		        ixx="1e-6" ixy="0.0" ixz="0.0"
+		        iyy="1e-6" iyz="0.0"
+		        izz="1e-6"
+		      />
+		</inertial>
+		<visual>
+			<origin xyz="0 0 0" rpy="0 0 0"/>
+			<geometry>
+				<mesh filename="package://ashwini/meshes/hokuyo.dae"/>
+			</geometry>
+		</visual>
+		<collision>
+			<origin xyz="0 0 0" rpy="0 0 0"/>
+			<geometry>
+				<box size="0.1 0.1 0.1"/>
+			</geometry>
+		</collision>
+	</link>
+  <joint name="camera_joint" type="fixed">
+		<origin xyz="0.006 -0.2 0.4" rpy="0 0.2 0" />
+		<parent link="base_link"/>
+		<child link="camera" />
+		<axis xyz="0 1 0"/>
+	</joint>
+	<!-- Hokoyu Joint -->
+	<joint name="hokuyo_joint" type="fixed">
+	    <origin xyz="0.001 -0.2 0.2" rpy="0 0 0" />
+	    <parent link="base_link"/>
+	    <child link="hokuyo" />
+	    <axis xyz="0 1 0"/>
+	</joint>
+    <!-- IMU Sensor -->
+  <link name="imu_link">
+    <inertial>
+      <mass value="0.05"/>
+      <origin xyz="0 0 0" rpy="0 0 0"/>
+      <inertia ixx="0.0001" ixy="0.0" ixz="0.0"
+               iyy="0.0001" iyz="0.0"
+               izz="0.0001"/>
+    </inertial>
+    <visual>
+      <geometry>
+        <box size="0.05 0.05 0.02"/>
+      </geometry>
+      <material name="Blue">
+        <color rgba="0.0 0.0 1.0 1.0"/>
+      </material>
+    </visual>
+    <collision>
+      <geometry>
+        <box size="0.05 0.05 0.02"/>
+      </geometry>
+    </collision>
+  </link>
+  <!-- IMU Joint (Attach to Base Link) -->
+  <joint name="imu_joint" type="fixed">
+    <parent link="base_link"/>
+    <child link="imu_link"/>
+    <origin xyz="-0.2 -0.2 0.144" rpy="0 0 0"/>
+  </joint>
 </robot>

Commit message: object avoidance with waypoint navigation

File: src/ashwini/urdf/ashwini.xacro (robot description, xacro)
@@ -2,11 +2,4 @@
 <robot name="ashwini" xmlns:xacro="ashwini_description_xacro_namespace">
   <!-- Dummy root link without inertia -->
-  <link name="dummy_root">
-  </link>
-  <joint name="dummy_root_to_base" type="fixed">
-    <parent link="dummy_root"/>
-    <child link="base_link"/>
-    <origin xyz="0 0 0" rpy="0 0 0"/>
-  </joint>
   <xacro:include filename="$(find ashwini)/urdf/ashwini.gazebo" />
   <xacro:property name="pi" value="3.1415926535897931" />
